Commit message: Implementing test cases (WIP)

File: tests/tester_robot.urdf (robot description, URDF)
Before this commit: robot test_robot, 5 links, 4 joints
Joints:
- removed joint joint3
- added joint joint2: type prismatic, parent link2, child link3, origin xyz=1 0 0, axis 0 0 1, limit lower=0 upper=1 effort=100 velocity=1
